Commit message: Update with launch file, cleanup before adding RGB camera from assignment

File: arduinobot/install/arduinobot_description/share/arduinobot_description/urdf/arduinobot.urdf.xacro (robot description, xacro)
@@ -117,3 +117,20 @@
         <limit lower="0.0" upper= "${PI/2}" effort="${effort}" velocity="${velocity}"/>
     </joint>
+    <!-- Add RGB camera holder to robot, fixed on the baseplate-->
+     <link name="rgb_camera">
+        <visual>
+            <!-- Intstructor-->
+            <origin rpy="-1.57 0 -1.57" xyz="-0.1 0.125 0.15"/>
+            <!--  Mine
+            <origin xyz="-0.01 0.45 0.2" rpy="0 -0.5 1.57"/>-->
+            <geometry>
+                <mesh filename="package://arduinobot_description/meshes/pi_camera.STL" scale="0.01 0.01 0.01"/>
+            </geometry>
+        </visual>
+     </link>
+     <joint name="rgb_camera_joint" type="fixed">
+        <parent link="base_link"/>
+        <child link="rgb_camera"/>
+        <origin xyz="0 0.45 0.2" rpy="0 -0.5 1.57"/>
+     </joint>
 </robot>

Commit message: Update with launch file, Non working RGB camera on Jellyfish with Iron ROS

File: arduinobot/install/arduinobot_description/share/arduinobot_description/urdf/arduinobot.urdf.xacro (robot description, xacro)
@@ -4,6 +4,18 @@
     <xacro:property name="effort" value="30.0"/>
     <xacro:property name="velocity" value="10.0"/>
+    <xacro:macro name="default_inertial" params="mass">
+        <inertial>
+            <mass value="${mass}"/>
+            <!-- Identity matrix, inertia of link is the same-->
+            <inertia ixx="1.0" ixy="0.0" ixz="0.0"
+                    iyy="1.0" iyz="0.0"
+                    izz="1.0"/>
+        </inertial>
+    </xacro:macro>
     <link name="world"/>
+    <!-- Tag meaning visual is what is shown, the actual mesh. geometry is the shape, origin shows where is should be displayed
+        from, collision and inertia are for simulation in gazebo-->
     <link name="base_link">
+        <xacro:default_inertial mass="1.0" />
         <visual>
             <!-- originally xyz set to 0 0 0. For all STL need to play with the values to make it centered
@@ -14,4 +26,10 @@
         </geometry>
         </visual>
+        <collision>
+            <origin rpy="0 0 0" xyz="-0.5 -0.5 0"/>
+        <geometry>
+            <mesh filename="package://arduinobot_description/meshes/basement.STL" scale="0.01 0.01 0.01"/>
+        </geometry>
+        </collision>
     </link>
     <joint name="virtual_joint" type="fixed">
@@ -21,4 +39,5 @@
     </joint>
     <link name="base_plate">
+        <xacro:default_inertial mass="0.1" />
         <visual>
             <origin rpy="0 0 0" xyz=" -0.39 -0.39 -0.56"/>
@@ -27,4 +46,10 @@
             </geometry>
         </visual>
+        <collision>
+            <origin rpy="0 0 0" xyz=" -0.39 -0.39 -0.56"/>
+            <geometry>
+                <mesh filename="package://arduinobot_description/meshes/base_plate.STL" scale="0.01 0.01 0.01"/>
+            </geometry>
+        </collision>
     </link>
     <!--
@@ -42,4 +67,5 @@
     <!-- Link for the rest of the bot- above was for base and main rotation-->
      <link name="forward_drive_arm">
+        <xacro:default_inertial mass="0.1" />
         <visual>
             <origin rpy="0 -${PI/2} ${PI/2}" xyz="0.19 0.06 -0.06"/>
@@ -48,4 +74,10 @@
             </geometry>
         </visual>
+        <collision>
+            <origin rpy="0 -${PI/2} ${PI/2}" xyz="0.19 0.06 -0.06"/>
+            <geometry>
+                <mesh filename="package://arduinobot_description/meshes/forward_drive_arm.STL" scale="0.01 0.01 0.01"/>
+            </geometry>
+        </collision>
      </link>
      <!-- Define the second joint for the bot-->
@@ -58,4 +90,5 @@
     </joint>
     <link name="horizontal_arm">
+        <xacro:default_inertial mass="0.1" />
         <visual>
             <origin rpy="${PI/2} 0 ${PI/2}" xyz="-0.03 -0.4 -0.06"/>
@@ -64,4 +97,10 @@
             </geometry>
         </visual>
+        <collision>
+            <origin rpy="${PI/2} 0 ${PI/2}" xyz="-0.03 -0.4 -0.06"/>
+            <geometry>
+                <mesh filename="package://arduinobot_description/meshes/horizontal_arm.STL" scale="0.01 0.01 0.01"/>
+            </geometry>
+        </collision>
     </link>
     <joint name="joint_3" type="revolute">
@@ -74,4 +113,5 @@
     <!--  claw Support link and Joint and stuff. I drank a two sangria this better work-->
     <link name="claw_arm">
+        <xacro:default_inertial mass="0.05" />
         <visual>
             <origin rpy="0 0 ${PI/2}" xyz="0 -0.05 -0.15"/>
@@ -80,4 +120,10 @@
             </geometry>
         </visual>
+        <collision>
+            <origin rpy="0 0 ${PI/2}" xyz="0 -0.05 -0.15"/>
+            <geometry>
+                <mesh filename="package://arduinobot_description/meshes/claw_support.STL" scale="0.01 0.01 0.01"/>
+            </geometry>
+        </collision>
     </link>
     <joint name="horizontal_arm_to_claw" type="fixed">
@@ -87,4 +133,5 @@
     </joint>
     <link name="gripper_right">
+        <xacro:default_inertial mass="0.01" />
         <visual>
             <origin xyz="-0.1 0.5 -0.1" rpy="0 0 -${PI/2}"/>
@@ -93,6 +140,13 @@
             </geometry>
         </visual>
+        <collision>
+            <origin xyz="-0.1 0.5 -0.1" rpy="0 0 -${PI/2}"/>
+            <geometry>
+                <mesh filename="package://arduinobot_description/meshes/right_finger.STL" scale="0.01 0.01 0.01" />
+            </geometry>
+        </collision>
     </link>
     <link name="gripper_left">
+        <xacro:default_inertial mass="0.01" />
         <visual>
             <origin xyz="-0.04 0.5 -0.1" rpy="0 0 -${PI/2}"/>
@@ -101,4 +155,10 @@
             </geometry>
         </visual>
+        <collision>
+            <origin xyz="-0.04 0.5 -0.1" rpy="0 0 -${PI/2}"/>
+            <geometry>
+                <mesh filename="package://arduinobot_description/meshes/left_finger.STL" scale="0.01 0.01 0.01" />
+            </geometry>
+        </collision>
     </link>
     <joint name="joint_4" type="revolute">
@@ -119,4 +179,5 @@
     <!-- Add RGB camera holder to robot, fixed on the baseplate-->
      <link name="rgb_camera">
+        <xacro:default_inertial mass="0.001"/>
         <visual>
             <!-- Intstructor-->
@@ -128,4 +189,12 @@
             </geometry>
         </visual>
+        <collision>
+            <origin rpy="-1.57 0 -1.57" xyz="-0.1 0.125 0.15"/>
+            <!--  Mine
+            <origin xyz="-0.01 0.45 0.2" rpy="0 -0.5 1.57"/>-->
+            <geometry>
+                <mesh filename="package://arduinobot_description/meshes/pi_camera.STL" scale="0.01 0.01 0.01"/>
+            </geometry>
+        </collision>
      </link>
      <joint name="rgb_camera_joint" type="fixed">
@@ -134,3 +203,4 @@
         <origin xyz="0 0.45 0.2" rpy="0 -0.5 1.57"/>
      </joint>
+     <!-- Gazebo for the camera-->
 </robot>

Commit message: Update with launch file, Non working controller manager.

File: arduinobot/install/arduinobot_description/share/arduinobot_description/urdf/arduinobot.urdf.xacro (robot description, xacro)
@@ -1,4 +1,6 @@
 <?xml version="1.0"?>
 <robot xmlns:xacro="http://www.ros.org/wiki/xacro" name="arduinobot">
+    <xacro:include filename="$(find arduinobot_description)/urdf/arduinobot_gazebo.xacro"/>
+    <xacro:include filename="$(find arduinobot_description)/urdf/arduinobot_ros2_control.xacro"/>
     <xacro:property name="PI" value="3.14159"/>
     <xacro:property name="effort" value="30.0"/>
@@ -13,4 +15,15 @@
         </inertial>
     </xacro:macro>
+    <!-- Gazebo and transmission for joints-->
+    <xacro:macro name="default_trans" params="number">
+        <transmission name="transmission_${number}">
+            <actuator name="moter_${number}" role="actuator1" />
+            <plugin>transmission_interface/SimpleTransmission</plugin>
+            <joint name="joint_${number}" role="joint1">
+                <!-- one degree of rotation correspondes to one degree of arm rotation-->
+                <mechanical_reduction>1.0</mechanical_reduction>
+            </joint>
+        </transmission>
+    </xacro:macro>
     <link name="world"/>
     <!-- Tag meaning visual is what is shown, the actual mesh. geometry is the shape, origin shows where is should be displayed
@@ -203,4 +216,8 @@
         <origin xyz="0 0.45 0.2" rpy="0 -0.5 1.57"/>
      </joint>
+     <xacro:default_trans number="1"/>
+     <xacro:default_trans number="2"/>
+     <xacro:default_trans number="3"/>
+     <xacro:default_trans number="4"/>
      <!-- Gazebo for the camera-->
 </robot>

File: arduinobot/install/arduinobot_description/share/arduinobot_description/urdf/arduinobot_gazebo.xacro (robot description, xacro)
@@ -6,38 +6,7 @@
         <robot_param>robot_description</robot_param>
         <robot_param_node>robot_state_publisher</robot_param_node>
+        <!-- File that contains config params for ros2 control library-->
         <parameters>$(find arduinobot_controller)/config/arduinobot_controllers.yaml</parameters>
       </plugin>
     </gazebo>
-    <gazebo reference="camera_link">
-        <sensor type="camera" name="rgb_camera">
-            <always_on>true</always_on>
-            <update_rate>30.0</update_rate>
-            <camera name="rgb_camera">
-                <horizontal_fov>1.15</horizontal_fov>
-                <vertical_fov>0.71</vertical_fov>
-                <image>
-                    <width>2304</width>
-                    <height>1296</height>
-                    <format>R8G8B8</format>
-                </image>
-                <distortion>
-                    <k1>0.0</k1>
-                    <k2>0.0</k2>
-                    <k3>0.0</k3>
-                    <p1>0.0</p1>
-                    <p2>0.0</p2>
-                    <center>0.5 0.5</center>
-                </distortion>
-            </camera>
-            <plugin name="camera_controller" filename="libgazebo_ros_camera.so">
-                <ros>
-                    <remapping>~/image_raw:=image_raw</remapping>
-                    <remapping>~/camera_info:=camera_info</remapping>
-                </ros>
-                <camera_name>rgb_camera</camera_name>
-                <frame_name>rgb_camera</frame_name>
-                <hack_baseline>0.2</hack_baseline>
-            </plugin>
-        </sensor>
-      </gazebo>
 </robot>
